Commit message: minor fix sensors path

File: rb1_description/urdf/sensors/all_sensors.urdf.xacro (robot description, xacro)
@@ -2,8 +2,8 @@
 <robot name="all_sensors" xmlns:xacro="http://www.ros.org/wiki/xacro">
   <!-- Imu -->
-  <xacro:include filename="$(find rover_description)/urdf/sensors/imu.urdf.xacro" />
+  <xacro:include filename="$(find rb1_description)/urdf/sensors/imu.urdf.xacro" />
   <!-- Hokuyo -->
-  <xacro:include filename="$(find rover_description)/urdf/sensors/hokuyo.urdf.xacro" />
+  <xacro:include filename="$(find rb1_description)/urdf/sensors/hokuyo.urdf.xacro" />
   <!-- Hokuyo -->
-  <xacro:include filename="$(find rover_description)/urdf/sensors/asus_xtion.urdf.xacro" />
+  <xacro:include filename="$(find rb1_description)/urdf/sensors/asus_xtion.urdf.xacro" />
 </robot>

File: rb1_description/urdf/sensors/asus_xtion.urdf.xacro (robot description, xacro)
@@ -13,5 +13,5 @@
         <origin rpy="${math_pi_over_2} 0 ${math_pi_over_2}" xyz="0 0 0"/>
         <geometry>
-          <mesh filename="package://rover_description/meshes/sensors/asus_xtion/asus_xtion_pro_live.dae" scale="0.001 0.001 0.001"/>
+          <mesh filename="package://rb1_description/meshes/sensors/asus_xtion/asus_xtion_pro_live.dae" scale="0.001 0.001 0.001"/>
         </geometry>
       </visual>
@@ -19,5 +19,5 @@
         <origin rpy="${math_pi_over_2} 0 ${math_pi_over_2}" xyz="0 0 0"/>
         <geometry>
-          <mesh filename="package://rover_description/meshes/sensors/asus_xtion/asus_xtion_pro_live.dae" scale="0.001 0.001 0.001"/>
+          <mesh filename="package://rb1_description/meshes/sensors/asus_xtion/asus_xtion_pro_live.dae" scale="0.001 0.001 0.001"/>
         </geometry>
       </collision>

File: rb1_description/urdf/sensors/hokuyo.urdf.xacro (robot description, xacro)
@@ -17,5 +17,5 @@
         <origin xyz="0 0 -0.05" rpy="0 0 0"/>
         <geometry>
-            <mesh filename="package://rover_description/meshes/sensors/hokuyo/hokuyo_ust_20lx.dae"/>
+            <mesh filename="package://rb1_description/meshes/sensors/hokuyo/hokuyo_ust_20lx.dae"/>
         </geometry>
       </visual>
