Commit message: initial files to change to ignition

File: rb1_description/robots/rb1_robot.urdf.xacro (robot description, xacro)
@@ -24,7 +24,68 @@
    </joint>
   <!-- Conollers -->
+  <ros2_control name="IgnitionSystem" type="system">
+    <hardware>
+      <plugin>ign_ros2_control/IgnitionSystem</plugin>
+    </hardware>
+    <joint name="left_wheel_joint">
+      <command_interface name="velocity">
+        <param name="min">-1</param>
+        <param name="max">1</param>
+      </command_interface>
+      <state_interface name="position"/>
+      <state_interface name="velocity"/>
+    </joint>
+    <joint name="right_wheel_joint">
+      <command_interface name="velocity">
+        <param name="min">-1</param>
+        <param name="max">1</param>
+      </command_interface>
+      <state_interface name="position"/>
+      <state_interface name="velocity"/>
+    </joint>
+    <joint name="j1_torso">
+      <command_interface name="position">
+        <param name="min">0</param>
+        <param name="max">0.36</param>
+      </command_interface>
+      <state_interface name="position">
+        <param name="initial_value">0.0</param>
+      </state_interface>
+      <state_interface name="velocity"/>
+      <state_interface name="effort"/>
+    </joint>
+    <joint name="j1_head">
+      <command_interface name="position">
+        <param name="min">-3.14159</param>
+        <param name="max">3.14159</param>
+      </command_interface>
+      <state_interface name="position">
+        <param name="initial_value">0.0</param>
+      </state_interface>
+      <state_interface name="velocity"/>
+      <state_interface name="effort"/>
+    </joint>
+    <joint name="j2_head">
+      <command_interface name="position">
+        <param name="min">-3.14159</param>
+        <param name="max">3.14159</param>
+      </command_interface>
+      <state_interface name="position">
+        <param name="initial_value">0.0</param>
+      </state_interface>
+      <state_interface name="velocity"/>
+      <state_interface name="effort"/>
+    </joint>
+  </ros2_control>
   <gazebo>
-    <plugin filename="libgazebo_ros2_control.so" name="gazebo_ros2_control">
+    <plugin filename="libign_ros2_control-system.so" name="ign_ros2_control::IgnitionROS2ControlPlugin">
       <parameters>$(find rb1_description)/config/rb1_control.yaml</parameters>
+      <ros>
+        <remapping>~/cmd_vel_unstamped:=cmd_vel</remapping>
+        <remapping>~/odom:=odom</remapping>
+        <remapping>/tf:=tf</remapping>
+        <remapping>/tf_static:=tf_static</remapping>
+        <remapping>/diagnostics:=diagnostics</remapping>
+      </ros>
     </plugin>
   </gazebo>

File: rb1_description/urdf/bases/base.gazebo.xacro (robot description, xacro)
@@ -12,29 +12,4 @@
 along with this program.  If not, see <https://www.gnu.org/licenses/>. -->
 <robot xmlns:xacro="http://www.ros.org/wiki/xacro">
-    <gazebo>
-        <plugin name='diff_base_controller' filename='libgazebo_ros_diff_drive.so'>
-            <ros>
-                <remapping>odom:=/robotnik_base_control/odom</remapping>
-            </ros>
-            <update_rate>100</update_rate>
-            <always_on>true</always_on>
-            <!-- wheels -->
-            <left_joint>left_wheel_joint</left_joint>
-            <right_joint>right_wheel_joint</right_joint>
-            <!-- kinematics -->
-            <wheel_separation>0.433</wheel_separation>
-            <wheel_diameter>0.152</wheel_diameter>
-            <!-- limits -->
-            <max_wheel_torque>20</max_wheel_torque>
-            <max_wheel_acceleration>1.0</max_wheel_acceleration>
-            <!-- output -->
-            <publish_odom>true</publish_odom>
-            <publish_odom_tf>true</publish_odom_tf>
-            <publish_wheel_tf>true</publish_wheel_tf>
-            <odometry_topic>odom</odometry_topic>
-            <odometry_frame>odom</odometry_frame>
-            <robot_base_frame>base_footprint</robot_base_frame>
-        </plugin>
-    </gazebo>
    <xacro:macro name="gazebo_colors" params="prefix">
         <gazebo reference="base_footprint">

File: rb1_description/urdf/torsos/torso_3dof.gazebo.xacro (robot description, xacro)
@@ -12,43 +12,5 @@
 along with this program.  If not, see <https://www.gnu.org/licenses/>. -->
 <robot xmlns:xacro="http://www.ros.org/wiki/xacro">
-  <ros2_control name="GazeboSystem" type="system">
-    <hardware>
-      <plugin>gazebo_ros2_control/GazeboSystem</plugin>
-    </hardware>
-    <joint name="j1_torso">
-      <command_interface name="position">
-        <param name="min">0</param>
-        <param name="max">0.36</param>
-      </command_interface>
-      <state_interface name="position">
-        <param name="initial_value">0.0</param>
-      </state_interface>
-      <state_interface name="velocity"/>
-      <state_interface name="effort"/>
-    </joint>
-    <joint name="j1_head">
-      <command_interface name="position">
-        <param name="min">-3.14159</param>
-        <param name="max">3.14159</param>
-      </command_interface>
-      <state_interface name="position">
-        <param name="initial_value">0.0</param>
-      </state_interface>
-      <state_interface name="velocity"/>
-      <state_interface name="effort"/>
-    </joint>
-    <joint name="j2_head">
-      <command_interface name="position">
-        <param name="min">-3.14159</param>
-        <param name="max">3.14159</param>
-      </command_interface>
-      <state_interface name="position">
-        <param name="initial_value">0.0</param>
-      </state_interface>
-      <state_interface name="velocity"/>
-      <state_interface name="effort"/>
-    </joint>
-  </ros2_control>
-  <gazebo>
+  <!-- <gazebo>
     <plugin name="rb1_torso_joint_state" filename="libgazebo_ros_joint_state_publisher.so">
       <update_rate>30</update_rate>
@@ -57,5 +19,5 @@
       <joint_name>j1_torso</joint_name>
     </plugin>
-  </gazebo>
+  </gazebo> -->
   <gazebo reference="torso_front_link">
     <selfCollide>true</selfCollide>
